Commit message: update urdf

File: src/curobo/content/assets/robot/frank_right_closed_description/frank_right_closed/frank_right_closed.urdf (robot description, URDF)
Before this commit: robot frank, 48 links, 47 joints
Links:
- added link World
- link base_link: geometry collision mesh filename=meshes/base_link_collisions_mesh_0.obj scale=1. 1. 1.; collision mesh filename=meshes/base_link_collisions_mesh_1.obj scale=1. 1. 1.
- link ewellix_lift_top_link: geometry collision mesh filename=meshes/ewellix_lift_top_link_collisions.obj scale=0.001 0.001 0.001; visual mesh filename=meshes/ewellix_lift_top_link_collisions.obj scale=0.001 0.001 0.001
- link left_arm_left_finger_mount: geometry collision mesh filename=meshes/left_arm_left_finger_mount_collisions.obj scale=1. 1. 1.; visual mesh filename=meshes/left_arm_left_finger_mount_collisions.obj scale=1. 1. 1.
- link left_arm_left_fingertip: geometry collision mesh filename=meshes/left_arm_left_fingertip_collisions.obj scale=1. 1. 1.; visual mesh filename=meshes/left_arm_left_fingertip_collisions.obj scale=1. 1. 1.
- link left_arm_left_inner_finger: geometry collision mesh filename=meshes/left_arm_left_inner_finger_collisions.obj scale=1. 1. 1.; visual mesh filename=meshes/left_arm_left_inner_finger_collisions.obj scale=1. 1. 1.
- link left_arm_left_inner_knuckle: geometry collision mesh filename=meshes/left_arm_left_inner_knuckle_collisions.obj scale=0.001 0.001 0.001; visual mesh filename=meshes/left_arm_left_inner_knuckle_collisions.obj scale=0.001 0.001 0.001
- link left_arm_left_outer_finger: geometry collision mesh filename=meshes/left_arm_left_outer_finger_collisions.obj scale=0.001 0.001 0.001; visual mesh filename=meshes/left_arm_left_outer_finger_collisions.obj scale=0.001 0.001 0.001
- link left_arm_left_outer_knuckle: geometry collision mesh filename=meshes/left_arm_left_outer_knuckle_collisions.obj scale=0.001 0.001 0.001; visual mesh filename=meshes/left_arm_left_outer_knuckle_collisions.obj scale=0.001 0.001 0.001
- link left_arm_right_finger_mount: geometry collision mesh filename=meshes/left_arm_right_finger_mount_collisions.obj scale=1. 1. 1.; visual mesh filename=meshes/left_arm_right_finger_mount_collisions.obj scale=1. 1. 1.
- link left_arm_right_fingertip: geometry collision mesh filename=meshes/left_arm_right_fingertip_collisions.obj scale=1. 1. 1.; visual mesh filename=meshes/left_arm_right_fingertip_collisions.obj scale=1. 1. 1.
- link left_arm_right_inner_finger: geometry collision mesh filename=meshes/left_arm_right_inner_finger_collisions.obj scale=1. 1. 1.; visual mesh filename=meshes/left_arm_right_inner_finger_collisions.obj scale=1. 1. 1.
- link left_arm_right_inner_knuckle: geometry collision mesh filename=meshes/left_arm_right_inner_knuckle_collisions.obj scale=0.001 0.001 0.001; visual mesh filename=meshes/left_arm_right_inner_knuckle_collisions.obj scale=0.001 0.001 0.001
- link left_arm_right_outer_finger: geometry collision mesh filename=meshes/left_arm_right_outer_finger_collisions.obj scale=0.001 0.001 0.001; visual mesh filename=meshes/left_arm_right_outer_finger_collisions.obj scale=0.001 0.001 0.001
- link left_arm_right_outer_knuckle: geometry collision mesh filename=meshes/left_arm_right_outer_knuckle_collisions.obj scale=0.001 0.001 0.001; visual mesh filename=meshes/left_arm_right_outer_knuckle_collisions.obj scale=0.001 0.001 0.001
- link left_arm_robotiq_arg2f_base_link: geometry collision mesh filename=meshes/left_arm_robotiq_arg2f_base_link_collisions.obj scale=1. 1. 1.; visual mesh filename=meshes/left_arm_robotiq_arg2f_base_link_collisions.obj scale=1. 1. 1.
- link left_base_link: geometry collision mesh filename=meshes/left_base_link_collisions.obj scale=1. 1. 1.; visual mesh filename=meshes/left_base_link_collisions.obj scale=1. 1. 1.
- link left_bracelet_link: geometry collision mesh filename=meshes/left_bracelet_link_collisions.obj scale=1. 1. 1.; visual mesh filename=meshes/left_bracelet_link_collisions.obj scale=1. 1. 1.
- link left_end_effector_link: mass None -> 0.000001
- link left_forearm_link: geometry collision mesh filename=meshes/left_forearm_link_collisions.obj scale=1. 1. 1.; visual mesh filename=meshes/left_forearm_link_collisions.obj scale=1. 1. 1.
- link left_half_arm_1_link: geometry collision mesh filename=meshes/left_half_arm_1_link_collisions.obj scale=1. 1. 1.; visual mesh filename=meshes/left_half_arm_1_link_collisions.obj scale=1. 1. 1.
- link left_half_arm_2_link: geometry collision mesh filename=meshes/left_half_arm_2_link_collisions.obj scale=1. 1. 1.; visual mesh filename=meshes/left_half_arm_2_link_collisions.obj scale=1. 1. 1.
- link left_shoulder_link: geometry collision mesh filename=meshes/left_shoulder_link_collisions.obj scale=1. 1. 1.; visual mesh filename=meshes/left_shoulder_link_collisions.obj scale=1. 1. 1.
- link left_spherical_wrist_1_link: geometry collision mesh filename=meshes/left_spherical_wrist_1_link_collisions.obj scale=1. 1. 1.; visual mesh filename=meshes/left_spherical_wrist_1_link_collisions.obj scale=1. 1. 1.
- link left_spherical_wrist_2_link: geometry collision mesh filename=meshes/left_spherical_wrist_2_link_collisions.obj scale=1. 1. 1.; visual mesh filename=meshes/left_spherical_wrist_2_link_collisions.obj scale=1. 1. 1.
- link left_tool_frame: mass None -> 0.000001
- link right_arm_left_finger_mount: geometry collision mesh filename=meshes/right_arm_left_finger_mount_collisions.obj scale=1. 1. 1.; visual mesh filename=meshes/right_arm_left_finger_mount_collisions.obj scale=1. 1. 1.
- link right_arm_left_fingertip: geometry collision mesh filename=meshes/right_arm_left_fingertip_collisions.obj scale=1. 1. 1.; visual mesh filename=meshes/right_arm_left_fingertip_collisions.obj scale=1. 1. 1.
- link right_arm_right_finger_mount: geometry collision mesh filename=meshes/right_arm_right_finger_mount_collisions.obj scale=1. 1. 1.; visual mesh filename=meshes/right_arm_right_finger_mount_collisions.obj scale=1. 1. 1.
- link right_arm_right_fingertip: geometry collision mesh filename=meshes/right_arm_right_fingertip_collisions.obj scale=1. 1. 1.; visual mesh filename=meshes/right_arm_right_fingertip_collisions.obj scale=1. 1. 1.
- link right_base_link: geometry collision mesh filename=meshes/right_base_link_collisions.obj scale=1. 1. 1.; visual mesh filename=meshes/right_base_link_collisions.obj scale=1. 1. 1.
- link right_bracelet_link: geometry collision mesh filename=meshes/right_bracelet_link_collisions.obj scale=1. 1. 1.; visual mesh filename=meshes/right_bracelet_link_collisions.obj scale=1. 1. 1.
- link right_end_effector_link: mass None -> 0.000001
- link right_forearm_link: geometry collision mesh filename=meshes/right_forearm_link_collisions.obj scale=1. 1. 1.; visual mesh filename=meshes/right_forearm_link_collisions.obj scale=1. 1. 1.
- link right_half_arm_1_link: geometry collision mesh filename=meshes/right_half_arm_1_link_collisions.obj scale=1. 1. 1.; visual mesh filename=meshes/right_half_arm_1_link_collisions.obj scale=1. 1. 1.
- link right_half_arm_2_link: geometry collision mesh filename=meshes/right_half_arm_2_link_collisions.obj scale=1. 1. 1.; visual mesh filename=meshes/right_half_arm_2_link_collisions.obj scale=1. 1. 1.
- link right_shoulder_link: geometry collision mesh filename=meshes/right_shoulder_link_collisions.obj scale=1. 1. 1.; visual mesh filename=meshes/right_shoulder_link_collisions.obj scale=1. 1. 1.
- link right_spherical_wrist_1_link: geometry collision mesh filename=meshes/right_spherical_wrist_1_link_collisions.obj scale=1. 1. 1.; visual mesh filename=meshes/right_spherical_wrist_1_link_collisions.obj scale=1. 1. 1.
- link right_spherical_wrist_2_link: geometry collision mesh filename=meshes/right_spherical_wrist_2_link_collisions.obj scale=1. 1. 1.; visual mesh filename=meshes/right_spherical_wrist_2_link_collisions.obj scale=1. 1. 1.
- link right_tool_frame: mass None -> 0.000001
Joints:
- added joint root_joint: type fixed, parent World, child base_link, origin xyz=0. 0. 0. rpy=0. 0. 0.
- joint left_arm_left_fingertip_fixed_joint: origin xyz=0.0184435 0.01721 0.0129684 rpy=1.5707964 0. 3.1415927 -> xyz=0.0184435 0.01721 0.0129684 rpy=1.5707964 0. -3.1415925
- joint left_arm_left_inner_knuckle_finger_joint: origin xyz=-0.0000052 -0.0682011 0.0979099 rpy=-0. 0. 3.1415052 -> xyz=-0.0000052 -0.0682011 0.0979099 rpy=0. 0. 3.1415052
- joint left_arm_left_inner_knuckle_joint: origin xyz=-0. -0. 0. rpy=-0. 0. -0.0000066 -> xyz=0. 0. 0. rpy=0. 0. -0.0000066
- joint left_arm_left_outer_finger_joint: origin xyz=0.0000019 -0.0621011 0.0508099 rpy=-0. 0. 3.1415055 -> xyz=0.0000019 -0.0621011 0.0508099 rpy=0. 0. 3.1415055
- joint left_arm_left_outer_knuckle_joint: origin xyz=-0. -0. 0. rpy=-0. 0. -0.0000066 -> xyz=0. 0. 0. rpy=0. 0. -0.0000066
- joint left_arm_right_fingertip_fixed_joint: origin xyz=0.0183902 0.01721 0.0129937 rpy=1.5707964 0. -3.1415927 -> xyz=0.0183902 0.01721 0.0129937 rpy=1.5707964 0. 3.1415925
- joint left_arm_right_inner_knuckle_joint: origin xyz=-0. -0. 0. rpy=-0. 0. -0.0000066 -> xyz=0. 0. 0. rpy=0. 0. -0.0000066
- joint left_arm_right_outer_finger_joint: origin xyz=-0.0000045 0.0621011 0.05081  rpy=0. -0. 0. -> xyz=-0.0000045 0.0621011 0.05081  rpy=0. 0. 0.
- joint left_arm_right_outer_knuckle_joint: origin xyz=-0. -0. 0. rpy=-0. 0. -0.0000066 -> xyz=0. 0. 0. rpy=0. 0. -0.0000066
- joint left_end_effector: origin xyz=-0.0615251 0.0000052 0.  rpy=3.1415927 0. -0.0000037 -> xyz=-0.0615251 0.0000052 0.  rpy=-3.1415925 0. -0.0000037
- joint left_joint_1: limit lower=-5.9999997 upper=5.9999997 effort=39. velocity=1.3963 -> lower=-5.9999991 upper=5.9999991 effort=39. velocity=1.3963
- joint left_joint_2: limit lower=-2.4099999 upper=2.4099999 effort=39. velocity=1.3963 -> lower=-2.4099997 upper=2.4099997 effort=39. velocity=1.3963
- joint left_joint_3: limit lower=-5.9999997 upper=5.9999997 effort=39. velocity=1.3963 -> lower=-5.9999991 upper=5.9999991 effort=39. velocity=1.3963; origin xyz=-0.0063793 -0.21038 0.  rpy=0. -0. 1.5708035 -> xyz=-0.0063793 -0.21038 0.  rpy=0. 0. 1.5708035
- joint left_joint_4: limit lower=-2.6599999 upper=2.6599999 effort=39. velocity=1.3963 -> lower=-2.6599997 upper=2.6599997 effort=39. velocity=1.3963; origin xyz=-0.21038 0.0063708 0.  rpy=0. -0. -1.5708035 -> xyz=-0.21038 0.0063708 0.  rpy=0. 0. -1.5708035
- joint left_joint_5: limit lower=-5.9999997 upper=5.9999997 effort=9. velocity=1.2218 -> lower=-5.9999991 upper=5.9999991 effort=9. velocity=1.2218
- joint left_joint_7: limit lower=-5.9999997 upper=5.9999997 effort=9. velocity=1.2218 -> lower=-5.9999991 upper=5.9999991 effort=9. velocity=1.2218; origin xyz=-0.0001696 -0.10593 0.  rpy=0. -0. 1.5708035 -> xyz=-0.0001696 -0.10593 0.  rpy=0. 0. 1.5708035
- joint left_tool_frame_joint: origin xyz=-0.1199949 0. -0.  rpy=0.0000001 -1.57 -0.0000001 -> xyz=-0.1199949 0. 0.  rpy=0.0000001 -0.0000001 -0.0000001
- joint right_arm_left_finger_joint: origin xyz=-0. 0. 0. rpy=0. -0. 0.0000002 -> xyz=0. 0. 0. rpy=0. 0. 0.0000002
- joint right_arm_left_inner_finger_joint: origin xyz=0. 0. 0. rpy=0. -0. -0.0000002 -> xyz=0. 0. 0. rpy=0. 0. -0.0000002
- joint right_arm_right_fingertip_fixed_joint: origin xyz=-0. 0.0000001 -0.0000001 rpy=0. 0. 0. -> xyz=0. 0.0000001 -0.0000001 rpy=0. 0. 0.
- joint right_end_effector: origin xyz=-0.0615251 0.0000051 0.  rpy=-3.1415927 0. -0.0000037 -> xyz=-0.0615251 0.0000051 0.  rpy=3.1415925 0. -0.0000037
- joint right_joint_1: limit lower=-5.9999997 upper=5.9999997 effort=39. velocity=1.3963 -> lower=-5.9999991 upper=5.9999991 effort=39. velocity=1.3963
- joint right_joint_2: limit lower=-2.4099999 upper=2.4099999 effort=39. velocity=1.3963 -> lower=-2.4099997 upper=2.4099997 effort=39. velocity=1.3963; origin xyz=-0.12838 0.0053741 -0.  rpy=0. -0. -1.5707927 -> xyz=-0.12838 0.0053741 0.  rpy=0. 0. -1.5707927
- joint right_joint_3: limit lower=-5.9999997 upper=5.9999997 effort=39. velocity=1.3963 -> lower=-5.9999991 upper=5.9999991 effort=39. velocity=1.3963; origin xyz=-0.0063792 -0.21038 0.  rpy=0. -0. 1.5708035 -> xyz=-0.0063792 -0.21038 0.  rpy=0. 0. 1.5708035
- joint right_joint_4: limit lower=-2.6599999 upper=2.6599999 effort=39. velocity=1.3963 -> lower=-2.6599997 upper=2.6599997 effort=39. velocity=1.3963
- joint right_joint_5: limit lower=-5.9999997 upper=5.9999997 effort=9. velocity=1.2218 -> lower=-5.9999991 upper=5.9999991 effort=9. velocity=1.2218; origin xyz=-0.0063793 -0.20843 0.  rpy=0. -0. 1.5708035 -> xyz=-0.0063793 -0.20843 0.  rpy=0. 0. 1.5708035
- joint right_joint_7: limit lower=-5.9999997 upper=5.9999997 effort=9. velocity=1.2218 -> lower=-5.9999991 upper=5.9999991 effort=9. velocity=1.2218; origin xyz=-0.0001696 -0.10593 0.  rpy=0. -0. 1.5708035 -> xyz=-0.0001696 -0.10593 0.  rpy=0. 0. 1.5708035
- joint right_kinova_joint_1: origin xyz=0. -0. 0. rpy=0.0000001 0. 0.  -> xyz=0. 0. 0. rpy=0.0000001 0. 0. 
- joint right_tool_frame_joint: origin xyz=-0.1199949 0. 0.  rpy=1.5707964 0 -1.5707963 -> xyz=-0.1199949 0. 0.  rpy=3.14 0. 0. 
